Commit message: first version of the hand

File: bin/demo1/resources/hand.urdf (robot description, URDF)
Before this commit: robot hand3finger, 8 links, 7 joints
Links:
- added link finger0-link0, mass 0.0716; visual box size=0.036 0.036 0.036
- added link finger0-link1, mass 0.0716; visual box size=0.016 0.015 0.025
- added link finger0-link2, mass 0.0509; visual box size=0.05 0.0168 0.025
- added link finger0-link3, mass 0.047; collision sphere radius=0.014; visual box size=0.0367 0.028 0.025
- added link finger1-link1, mass 0.0716; visual box size=0.054 0.028 0.025
- added link finger1-link2, mass 0.0509; visual box size=0.0384 0.028 0.025
- added link finger1-link3, mass 0.047; collision sphere radius=0.014; visual box size=0.0187 0.028 0.025
- added link finger2-link0, mass 0.0716; visual box size=0.016 0.028 0.025
- added link finger2-link1, mass 0.0716; visual box size=0.054 0.028 0.025
- added link finger2-link2, mass 0.0509; visual box size=0.0384 0.028 0.025
- added link finger2-link3, mass 0.047; collision sphere radius=0.014; visual box size=0.0187 0.028 0.025
- added link finger3-link0, mass 0.0716; visual box size=0.016 0.028 0.025
- added link finger3-link1, mass 0.0716; visual box size=0.054 0.028 0.025
- added link finger3-link2, mass 0.0509; visual box size=0.0384 0.028 0.025
- added link finger3-link3, mass 0.047; collision sphere radius=0.014; visual box size=0.0187 0.028 0.025
- link finger1-link0: mass 0.08 -> 0.0716; geometry visual box size=0.016 0.028 0.025
- link palm: mass 0.3 -> 0.5; geometry visual box size=0.095 0.11 0.055
Joints:
- added joint finger0-j0: type revolute, parent palm, child finger0-link0, origin xyz=-0.0155 -0.015 0.008 rpy=0 0 0, axis 1 0 0, limit lower=-2.967 upper=2.967 effort=176 velocity=1.7104
- added joint finger0-j1: type revolute, parent finger0-link0, child finger0-link1, origin xyz=-0.01 -0.036 0 rpy=0 0 0, axis 0 1 0, limit lower=-2.967 upper=2.967 effort=176 velocity=1.7104
- added joint finger0-j2: type revolute, parent finger0-link1, child finger0-link2, origin xyz=0 -0.015 0 rpy=0 0 0, axis 0 0 1, limit lower=-2.967 upper=2.967 effort=176 velocity=1.7104
- added joint finger0-j3: type revolute, parent finger0-link2, child finger0-link3, origin xyz=0.05 0 0 rpy=0 0 0, axis 0 0 1, limit lower=-2.967 upper=2.967 effort=176 velocity=1.7104
- added joint finger1-j1: type revolute, parent finger1-link0, child finger1-link1, origin xyz=0.016 0 0 rpy=0 0 0, axis 0 1 0, limit lower=-2.967 upper=2.967 effort=176 velocity=1.7104
- added joint finger1-j2: type revolute, parent finger1-link1, child finger1-link2, origin xyz=0.054 0 0 rpy=0 0 0, axis 0 1 0, limit lower=-2.967 upper=2.967 effort=176 velocity=1.7104
- added joint finger1-j3: type revolute, parent finger1-link2, child finger1-link3, origin xyz=0.0384 0 0 rpy=0 0 0, axis 0 1 0, limit lower=-2.967 upper=2.967 effort=176 velocity=1.7104
- added joint finger2-j0: type revolute, parent palm, child finger2-link0, origin xyz=0.0475 0.0 -0.015 rpy=0 0 0, axis 1 0 0, limit lower=-2.967 upper=2.967 effort=176 velocity=1.7104
- added joint finger2-j1: type revolute, parent finger2-link0, child finger2-link1, origin xyz=0.016 0.0 0.0 rpy=0 0 0, axis 0 1 0, limit lower=-2.967 upper=2.967 effort=176 velocity=1.7104
- added joint finger2-j2: type revolute, parent finger2-link1, child finger2-link2, origin xyz=0.054 0 0 rpy=0 0 0, axis 0 1 0, limit lower=-2.967 upper=2.967 effort=176 velocity=1.7104
- added joint finger2-j3: type revolute, parent finger2-link2, child finger2-link3, origin xyz=0.0384 0 0 rpy=0 0 0, axis 0 1 0, limit lower=-2.967 upper=2.967 effort=176 velocity=1.7104
- added joint finger3-j0: type revolute, parent palm, child finger3-link0, origin xyz=0.0475 0.041 -0.015 rpy=0 0 0, axis 1 0 0, limit lower=-2.967 upper=2.967 effort=176 velocity=1.7104
- added joint finger3-j1: type revolute, parent finger3-link0, child finger3-link1, origin xyz=0.016 0 0 rpy=0 0 0, axis 0 1 0, limit lower=-2.967 upper=2.967 effort=176 velocity=1.7104
- added joint finger3-j2: type revolute, parent finger3-link1, child finger3-link2, origin xyz=0.054 0 0 rpy=0 0 0, axis 0 1 0, limit lower=-2.967 upper=2.967 effort=176 velocity=1.7104
- added joint finger3-j3: type revolute, parent finger3-link2, child finger3-link3, origin xyz=0.0384 0 0 rpy=0 0 0, axis 0 1 0, limit lower=-2.967 upper=2.967 effort=176 velocity=1.7104
- joint finger1-j0: axis 0 0 1 -> 1 0 0; origin xyz=0 0 0 rpy=1.5707 0 0 -> xyz=0.0475 -0.041 -0.015 rpy=0 0 0

File: resources/hand.urdf (robot description, URDF)
Before this commit: robot hand3finger, 8 links, 7 joints
Links:
- added link finger0-link0, mass 0.0716; visual box size=0.036 0.036 0.036
- added link finger0-link1, mass 0.01; visual box size=0.016 0.015 0.025
- added link finger0-link2, mass 0.0509; visual box size=0.05 0.0168 0.025
- added link finger0-link3, mass 0.047; collision sphere radius=0.014; visual box size=0.0367 0.028 0.025
- added link finger1-link1, mass 0.0716; visual box size=0.054 0.028 0.025
- added link finger1-link2, mass 0.0509; visual box size=0.0384 0.028 0.025
- added link finger1-link3, mass 0.047; collision sphere radius=0.014; visual box size=0.0187 0.028 0.025
- added link finger2-link0, mass 0.0716; visual box size=0.016 0.028 0.025
- added link finger2-link1, mass 0.0716; visual box size=0.054 0.028 0.025
- added link finger2-link2, mass 0.0509; visual box size=0.0384 0.028 0.025
- added link finger2-link3, mass 0.047; collision sphere radius=0.014; visual box size=0.0187 0.028 0.025
- added link finger3-link0, mass 0.0716; visual box size=0.016 0.028 0.025
- added link finger3-link1, mass 0.0716; visual box size=0.054 0.028 0.025
- added link finger3-link2, mass 0.0509; visual box size=0.0384 0.028 0.025
- added link finger3-link3, mass 0.047; collision sphere radius=0.014; visual box size=0.0187 0.028 0.025
- link finger1-link0: mass 0.08 -> 0.0716; geometry visual box size=0.016 0.028 0.025
- link palm: mass 0.3 -> 0.5; geometry visual box size=0.095 0.11 0.055
Joints:
- added joint finger0-j0: type revolute, parent palm, child finger0-link0, origin xyz=-0.0155 -0.015 0.008 rpy=0 0 0, axis 1 0 0, limit lower=-2.967 upper=2.967 effort=176 velocity=1.7104
- added joint finger0-j1: type revolute, parent finger0-link0, child finger0-link1, origin xyz=-0.01 -0.036 0 rpy=0 0 0, axis 0 1 0, limit lower=-2.967 upper=2.967 effort=176 velocity=1.7104
- added joint finger0-j2: type revolute, parent finger0-link1, child finger0-link2, origin xyz=0 -0.015 0 rpy=0 0 0, axis 0 0 1, limit lower=-2.967 upper=2.967 effort=176 velocity=1.7104
- added joint finger0-j3: type revolute, parent finger0-link2, child finger0-link3, origin xyz=0.05 0 0 rpy=0 0 0, axis 0 0 1, limit lower=-2.967 upper=2.967 effort=176 velocity=1.7104
- added joint finger1-j1: type revolute, parent finger1-link0, child finger1-link1, origin xyz=0.016 0 0 rpy=0 0 0, axis 0 1 0, limit lower=-2.967 upper=2.967 effort=176 velocity=1.7104
- added joint finger1-j2: type revolute, parent finger1-link1, child finger1-link2, origin xyz=0.054 0 0 rpy=0 0 0, axis 0 1 0, limit lower=-2.967 upper=2.967 effort=176 velocity=1.7104
- added joint finger1-j3: type revolute, parent finger1-link2, child finger1-link3, origin xyz=0.0384 0 0 rpy=0 0 0, axis 0 1 0, limit lower=-2.967 upper=2.967 effort=176 velocity=1.7104
- added joint finger2-j0: type revolute, parent palm, child finger2-link0, origin xyz=0.0475 0.0 -0.015 rpy=0 0 0, axis 1 0 0, limit lower=-2.967 upper=2.967 effort=176 velocity=1.7104
- added joint finger2-j1: type revolute, parent finger2-link0, child finger2-link1, origin xyz=0.016 0.0 0.0 rpy=0 0 0, axis 0 1 0, limit lower=-2.967 upper=2.967 effort=176 velocity=1.7104
- added joint finger2-j2: type revolute, parent finger2-link1, child finger2-link2, origin xyz=0.054 0 0 rpy=0 0 0, axis 0 1 0, limit lower=-2.967 upper=2.967 effort=176 velocity=1.7104
- added joint finger2-j3: type revolute, parent finger2-link2, child finger2-link3, origin xyz=0.0384 0 0 rpy=0 0 0, axis 0 1 0, limit lower=-2.967 upper=2.967 effort=176 velocity=1.7104
- added joint finger3-j0: type revolute, parent palm, child finger3-link0, origin xyz=0.0475 0.041 -0.015 rpy=0 0 0, axis 1 0 0, limit lower=-2.967 upper=2.967 effort=176 velocity=1.7104
- added joint finger3-j1: type revolute, parent finger3-link0, child finger3-link1, origin xyz=0.016 0 0 rpy=0 0 0, axis 0 1 0, limit lower=-2.967 upper=2.967 effort=176 velocity=1.7104
- added joint finger3-j2: type revolute, parent finger3-link1, child finger3-link2, origin xyz=0.054 0 0 rpy=0 0 0, axis 0 1 0, limit lower=-2.967 upper=2.967 effort=176 velocity=1.7104
- added joint finger3-j3: type revolute, parent finger3-link2, child finger3-link3, origin xyz=0.0384 0 0 rpy=0 0 0, axis 0 1 0, limit lower=-2.967 upper=2.967 effort=176 velocity=1.7104
- joint finger1-j0: axis 0 0 1 -> 1 0 0; origin xyz=0 0 0 rpy=1.5707 0 0 -> xyz=0.0475 -0.041 -0.015 rpy=0 0 0

Commit message: finished the initialize code

File: bin/demo1/resources/hand.urdf (robot description, URDF)
Before this commit: robot hand3finger, 23 links, 22 joints
Links:
- link finger0-link1: mass 0.0716 -> 0.01
Joints:
- joint finger0-j0: origin xyz=-0.0155 -0.015 0.008 rpy=0 0 0 -> xyz=-0.0155 -0.015 -0.008 rpy=0 0 0
- joint finger1-j1: origin xyz=0.016 0 0 rpy=0 0 0 -> xyz=0.016 0 0 rpy=0 0.3 0
- joint finger1-j2: origin xyz=0.054 0 0 rpy=0 0 0 -> xyz=0.054 0 0 rpy=0 0.3 0
- joint finger1-j3: origin xyz=0.0384 0 0 rpy=0 0 0 -> xyz=0.0384 0 0 rpy=0 0.3 0
- joint finger2-j1: origin xyz=0.016 0.0 0.0 rpy=0 0 0 -> xyz=0.016 0.0 0.0 rpy=0 0.3 0
- joint finger2-j2: origin xyz=0.054 0 0 rpy=0 0 0 -> xyz=0.054 0 0 rpy=0 0.3 0
- joint finger2-j3: origin xyz=0.0384 0 0 rpy=0 0 0 -> xyz=0.0384 0 0 rpy=0 0.3 0
- joint finger3-j0: limit lower=-2.967 upper=2.967 effort=176 velocity=1.7104 -> (none)
- joint finger3-j1: limit lower=-2.967 upper=2.967 effort=176 velocity=1.7104 -> (none); origin xyz=0.016 0 0 rpy=0 0 0 -> xyz=0.016 0 0 rpy=0 0.3 0
- joint finger3-j2: limit lower=-2.967 upper=2.967 effort=176 velocity=1.7104 -> (none); origin xyz=0.054 0 0 rpy=0 0 0 -> xyz=0.054 0 0 rpy=0 0.3 0
- joint finger3-j3: limit lower=-2.967 upper=2.967 effort=176 velocity=1.7104 -> (none); origin xyz=0.0384 0 0 rpy=0 0 0 -> xyz=0.0384 0 0 rpy=0 0.3 0

File: resources/hand.urdf (robot description, URDF)
Before this commit: robot hand3finger, 23 links, 22 joints
Joints:
- joint finger0-j0: origin xyz=-0.0155 -0.015 0.008 rpy=0 0 0 -> xyz=-0.0155 -0.015 -0.008 rpy=0 0 0
- joint finger1-j1: origin xyz=0.016 0 0 rpy=0 0 0 -> xyz=0.016 0 0 rpy=0 0.3 0
- joint finger1-j2: origin xyz=0.054 0 0 rpy=0 0 0 -> xyz=0.054 0 0 rpy=0 0.3 0
- joint finger1-j3: origin xyz=0.0384 0 0 rpy=0 0 0 -> xyz=0.0384 0 0 rpy=0 0.3 0
- joint finger2-j1: origin xyz=0.016 0.0 0.0 rpy=0 0 0 -> xyz=0.016 0.0 0.0 rpy=0 0.3 0
- joint finger2-j2: origin xyz=0.054 0 0 rpy=0 0 0 -> xyz=0.054 0 0 rpy=0 0.3 0
- joint finger2-j3: origin xyz=0.0384 0 0 rpy=0 0 0 -> xyz=0.0384 0 0 rpy=0 0.3 0
- joint finger3-j1: origin xyz=0.016 0 0 rpy=0 0 0 -> xyz=0.016 0 0 rpy=0 0.3 0
- joint finger3-j2: origin xyz=0.054 0 0 rpy=0 0 0 -> xyz=0.054 0 0 rpy=0 0.3 0
- joint finger3-j3: origin xyz=0.0384 0 0 rpy=0 0 0 -> xyz=0.0384 0 0 rpy=0 0.3 0

Commit message: An intermediate version while still a little bit bug in it

File: bin/demo1/resources/hand.urdf (robot description, URDF)
Before this commit: robot hand3finger, 23 links, 22 joints
Joints:
- joint finger0-j0: origin xyz=-0.0155 -0.015 -0.008 rpy=0 0 0 -> xyz=-0.0155 -0.015 -0.008 rpy=0.1 0 0
- joint finger0-j1: origin xyz=-0.01 -0.036 0 rpy=0 0 0 -> xyz=-0.01 -0.036 0 rpy=0 0.1 0
- joint finger0-j2: origin xyz=0 -0.015 0 rpy=0 0 0 -> xyz=0 -0.015 0 rpy=0 0 0.2
- joint finger0-j3: origin xyz=0.05 0 0 rpy=0 0 0 -> xyz=0.05 0 0 rpy=0 0 0.2
- joint finger3-j0: limit (none) -> lower=-2.967 upper=2.967 effort=176 velocity=1.7104
- joint finger3-j1: limit (none) -> lower=-2.967 upper=2.967 effort=176 velocity=1.7104
- joint finger3-j2: limit (none) -> lower=-2.967 upper=2.967 effort=176 velocity=1.7104
- joint finger3-j3: limit (none) -> lower=-2.967 upper=2.967 effort=176 velocity=1.7104

File: resources/hand.urdf (robot description, URDF)
Before this commit: robot hand3finger, 23 links, 22 joints
Joints:
- joint finger0-j0: origin xyz=-0.0155 -0.015 -0.008 rpy=0 0 0 -> xyz=-0.0155 -0.015 -0.008 rpy=0.1 0 0
- joint finger0-j1: origin xyz=-0.01 -0.036 0 rpy=0 0 0 -> xyz=-0.01 -0.036 0 rpy=0 0.1 0
- joint finger0-j2: origin xyz=0 -0.015 0 rpy=0 0 0 -> xyz=0 -0.015 0 rpy=0 0 0.2
- joint finger0-j3: origin xyz=0.05 0 0 rpy=0 0 0 -> xyz=0.05 0 0 rpy=0 0 0.2

Commit message: change the left-hand model into the right-hand model

File: bin/demo1/resources/hand.urdf (robot description, URDF)
Before this commit: robot hand3finger, 23 links, 22 joints
Links:
- link finger0-link1: geometry visual box size=0.016 0.018 0.025
Joints:
- joint finger0-j0: origin xyz=-0.0155 -0.015 -0.008 rpy=0.1 0 0 -> xyz=-0.0155 0.015 -0.008 rpy=0 0 -0.087
- joint finger0-j1: origin xyz=-0.01 -0.036 0 rpy=0 0.1 0 -> xyz=-0.01 0.036 0 rpy=0 0 0
- joint finger0-j2: origin xyz=0 -0.015 0 rpy=0 0 0.2 -> xyz=0 0.018 0 rpy=0 0 1.57
- joint finger0-j3: origin xyz=0.05 0 0 rpy=0 0 0.2 -> xyz=0.05 0 0 rpy=0 0 0
